File: hardware/gokart.kicad_pcb (KiCad board)
At the start: 2 copper layers, 100 x 60 mm, 116 parts, among them IC1 TPS54527, J1 USB, P1 BAT, P10 D5, P11 D3/SCL, P12 D2/SDA, P13 D4, P14 D6, P15 D7, P16 A4, P17 A3, P18 A2, P19 A1, P2 CONN_8, P20 A0, P21 12V, P22 5VA, P23 5V, P24 3.3V, P25 GND, P3 CONN_8, P4 ISP, P5 CONN_8, P6 CONN_8, P7 IO8, P8 IO9, P9 IO10, SW1 RESET, SW2 SW, T1 FDD4243, T2 FDD4243, U1 NCP1117ST33T3G, U10 ATmega32U4, U11 XBEE868, U12 FT232RL, U2 74HC595, U3 74HC595, U4 ULN2003, U5 ULN2003, U6 74HC595, U7 74HC595, U8 ULN2003, U9 ULN2003, X1 16MHz

Commit message: Updated hardware
Parts:
- removed P8: IO9, Pin_Headers:Pin_Header_Straight_1x01
- removed R20: 4k7, Resistors_SMD:R_0805
- removed R22: 10k, Resistors_SMD:R_0805
- removed SW2: SW, Discret:SW_PUSH_SMALL
- added D8: 1N4148W, My:SOD-123, F.Cu at (113.2, 81.7)
- IC1: footprint SMD_Packages:SSOP8-9 -> SMD_Packages:SOIC-8-N-1EP
- R10, R8: footprint Resistors_SMD:R_0805 -> SMD_Packages:SMD-0603
- SW1: footprint Discret:SW_PUSH_SMALL -> My:SW_PUSH_SMALL
- U12: footprint SMD_Packages:SO-28 -> SMD_Packages:SSOP-28
- moved R6 3.43 mm to (51.9, 74.8)
- moved C5 3.30 mm to (55.0, 75.3)
- moved C11 2.16 mm to (51.2, 71.2)
- moved C3 2.16 mm to (55.2, 72.3)
- moved R5 2.16 mm to (53.2, 71.4)
- moved IC1 1.35 mm to (60.3, 73.7)
- moved C30 0.97 mm to (58.5, 104.4)
Connections:
- U10 pad 29: /IO9 -> /XBEE_RES
- U12 pad 2: /DTR -> /XBEE_RES
Routing:
- net /XBEE_RES: track 0.00 -> 104.9 mm, vias 0 -> 2
- net /DTR: track 80.8 -> 0.00 mm, vias 2 -> 0
- net Net-(U11-Pad20): track 56.5 -> 0.00 mm, vias 1 -> 0
- net GND: track 598.7 -> 576.6 mm, vias 27 -> 25
- net Net-(D8-Pad1): track 0.00 -> 21.8 mm, vias 0 -> 1
- net /IO9: track 10.1 -> 0.00 mm
- net +5V: track 317.4 -> 326.4 mm
- net Net-(U11-Pad9): track 7.79 -> 0.38 mm
- net VUSB: track 68.6 -> 62.0 mm, vias 4 -> 6
- net /D1/TX: track 114.1 -> 108.2 mm
- net /D-: track 28.7 -> 32.8 mm
- net /D+: track 35.6 -> 39.5 mm
- net Net-(C33-Pad2): track 2.04 -> 5.40 mm
- net /RTS: track 78.1 -> 74.7 mm
- net /CTS: track 64.2 -> 66.9 mm
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Other:
- board text added: "gokart v2.0"
- board text removed: "gokart v1.0"
