File: hardware/gokart.sch (KiCad schematic (older format))
At the start: 112 parts, among them IC1 TPS54527, J1 USB, P1 BAT, P10 D5, P11 D3/SCL, P12 D2/SDA, P13 D4, P14 D6, P15 D7, P16 A4, P17 A3, P18 A2, P19 A1, P2 CONN_8, P20 A0, P21 12V, P22 5VA, P23 5V, P24 3.3V, P25 GND, P3 CONN_8, P4 ISP, P5 CONN_8, P6 CONN_8, P7 IO8, P8 IO9, P9 IO10, SW1 RESET, SW2 SW, T1 FDD4243, T2 FDD4243, U1 NCP1117ST33T3G, U10 ATmega32U4, U11 XBEE868, U12 FT232RL, U2 74HC595, U3 74HC595, U4 ULN2003, U5 ULN2003, U6 74HC595, U7 74HC595, U8 ULN2003, U9 ULN2003, X1 16MHz

Commit message: Updated hardware
Parts:
- removed P8: IO9, Pin_Headers:Pin_Header_Straight_1x01, symbol CONN_01X01
- removed R20: 4k7, Resistors_SMD:R_0805, symbol R_SMALL
- removed R22: 10k, Resistors_SMD:R_0805, symbol R_SMALL
- removed SW2: SW, Discret:SW_PUSH_SMALL, symbol SW_PUSH_MINI
- added D8: 1N4148W, My:SOD-123, symbol DIODE
- IC1: footprint SMD_Packages:SSOP8-9 -> SMD_Packages:SOIC-8-N-1EP
- R10, R8: footprint Resistors_SMD:R_0805 -> SMD_Packages:SMD-0603
- SW1: footprint Discret:SW_PUSH_SMALL -> My:SW_PUSH_SMALL
- U12: footprint SMD_Packages:SO-28 -> SMD_Packages:SSOP-28
Connections:
- net IO9 is gone; now on net XBEE_RES: U10.29 ((ADC12/OC1A/~OC4B~/PCINT12)PB5)
- net at U11.5 (NRESET): now also D8.1 (A)
- net DTR renamed XBEE_RES
- net XBEE_RES: now also D8.2 (K)
- no-connect marks 27 -> 28
